File: UV-Vis_Spectrometer_Photodiode_Breakout/UV-Vis_Spectrometer_Photodiode_Breakout.kicad_sch (KiCad schematic)
At the start: 48 parts, among them J1 Conn_01x05, J2 Conn_01x02, J3 Conn_01x02, Q1 BSS138BK,215, Q2 BSS138BK,215, Q3 BSS138BK,215, U1 TLV8811DBVR, U2 LM317BS-TR, U3 LTC2451

Commit message: Made footprint for photodiode. Made basic layout for PCB.
Parts:
- D1: footprint OptoDevice:Kodenshi_LG206D -> PhotoDiode_BPW21R:BPW21R
- D4: footprint LED_SMD:LED_Cree-XHP50_3V_HighDensity -> LED_SMD:LED_0603_1608Metric_Pad1.05x0.95mm_HandSolder
- D5: footprint Diode_SMD:D_0603_1608Metric_Pad1.05x0.95mm_HandSolder -> LED_SMD:LED_0603_1608Metric_Pad1.05x0.95mm_HandSolder
Changed lines of the file:
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@@
 			)
 		)
-		(property "Footprint" "LED_SMD:LED_Cree-XHP50_3V_HighDensity"
+		(property "Footprint" "LED_SMD:LED_0603_1608Metric_Pad1.05x0.95mm_HandSolder"
 			(at 220.98 143.51 0)
 			(hide yes)
@@
 			)
 		)
-		(property "Footprint" "OptoDevice:Kodenshi_LG206D"
+		(property "Footprint" "PhotoDiode_BPW21R:BPW21R"
 			(at 107.95 147.32 0)
 			(hide yes)
@@
 			)
 		)
-		(property "Footprint" "Diode_SMD:D_0603_1608Metric_Pad1.05x0.95mm_HandSolder"
+		(property "Footprint" "LED_SMD:LED_0603_1608Metric_Pad1.05x0.95mm_HandSolder"
 			(at 208.28 143.51 0)
 			(hide yes)

Commit message: Attempted to make layout smaller.
Parts:
- D2, D3: value 1N4001 -> CDSU101A; footprint Diode_THT:D_DO-41_SOD81_P10.16mm_Horizontal -> https://www.digikey.com/en/products/detail/comchip-technology/CDSU101A/1121034
Changed lines of the file:
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@@
 			)
 		)
-		(property "Value" "1N4001"
+		(property "Value" "CDSU101A"
 			(at 223.52 27.94 0)
 			(show_name no)
@@
 			)
 		)
-		(property "Footprint" "Diode_THT:D_DO-41_SOD81_P10.16mm_Horizontal"
+		(property "Footprint" "https://www.digikey.com/en/products/detail/comchip-technology/CDSU101A/1121034"
 			(at 223.52 31.75 0)
 			(hide yes)
@@
 			)
 		)
-		(property "Value" "1N4001"
+		(property "Value" "CDSU101A"
 			(at 251.46 41.9099 90)
 			(show_name no)
@@
 			)
 		)
-		(property "Footprint" "Diode_THT:D_DO-41_SOD81_P10.16mm_Horizontal"
+		(property "Footprint" "https://www.digikey.com/en/products/detail/comchip-technology/CDSU101A/1121034"
 			(at 248.92 40.64 0)
 			(hide yes)
