File: UV-Vis_Spectrometer_Photodiode_Breakout/UV-Vis_Spectrometer_Photodiode_Breakout.kicad_sch (KiCad schematic)
At the start: 48 parts, among them J1 Conn_01x05, J2 Conn_01x02, J3 Conn_01x02, Q1 BSS138BK,215, Q2 BSS138BK,215, Q3 BSS138BK,215, U1 TLV8811DBVR, U2 LM317BS-TR, U3 LTC2451

Commit message: Moved the layout around a bit.
Parts:
- D2, D3: footprint https://www.digikey.com/en/products/detail/comchip-technology/CDSU101A/1121034 -> Diode_SMD:D_0603_1608Metric_Pad1.05x0.95mm_HandSolder
Connections:
- net IN-: now reaches C1.1, C10.1, C11.1, D1.1 (K), R5.1, R6.1, R7.1, U1.3 (-)
Changed lines of the file:
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@@
 	(wire
 		(pts
+			(xy 107.95 143.51) (xy 129.54 143.51)
+		)
+		(stroke
+			(width 0)
+			(type default)
+		)
+	)
+	(wire
+		(pts
 			(xy 120.65 110.49) (xy 120.65 114.3)
 		)
@@
 	(wire
 		(pts
-			(xy 107.95 143.51) (xy 129.54 143.51)
-		)
-		(stroke
-			(width 0)
-			(type default)
-		)
-	)
-	(wire
-		(pts
 			(xy 248.92 63.5) (xy 234.95 63.5)
 		)
@@
 		)
 	)
+	(label "IN-"
+		(at 113.03 143.51 0)
+		(effects
+			(font
+				(size 1.27 1.27)
+			)
+			(justify left bottom)
+		)
+	)
 	(global_label "RR3+"
 		(shape output)
@@
 			)
 		)
-		(property "Footprint" "https://www.digikey.com/en/products/detail/comchip-technology/CDSU101A/1121034"
+		(property "Footprint" "Diode_SMD:D_0603_1608Metric_Pad1.05x0.95mm_HandSolder"
 			(at 223.52 31.75 0)
 			(hide yes)
@@
 			)
 		)
-		(property "Datasheet" "http://www.vishay.com/docs/88503/1n4001.pdf"
+		(property "Datasheet" "https://www.digikey.com/en/products/detail/comchip-technology/CDSU101A/1121034"
 			(at 223.52 31.75 0)
 			(hide yes)
@@
 			)
 		)
-		(property "Footprint" "https://www.digikey.com/en/products/detail/comchip-technology/CDSU101A/1121034"
+		(property "Footprint" "Diode_SMD:D_0603_1608Metric_Pad1.05x0.95mm_HandSolder"
 			(at 248.92 40.64 0)
 			(hide yes)
@@
 			)
 		)
-		(property "Datasheet" "http://www.vishay.com/docs/88503/1n4001.pdf"
+		(property "Datasheet" "https://www.digikey.com/en/products/detail/comchip-technology/CDSU101A/1121034"
 			(at 248.92 40.64 0)
 			(hide yes)

Commit message: Updated footprint for Reed Relays.
Parts:
- RR1, RR2, RR3: footprint Relay_THT:Relay_SPST_StandexMeder_SIL_Form1A -> UV_Vis_Library:Relay_SPDT_9007_05_00
Changed lines of the file:
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@@
 			)
 		)
-		(property "Footprint" "Relay_THT:Relay_SPST_StandexMeder_SIL_Form1A"
+		(property "Footprint" "UV_Vis_Library:Relay_SPDT_9007_05_00"
 			(at 135.89 68.58 0)
 			(hide yes)
@@
 			)
 		)
-		(property "Footprint" "Relay_THT:Relay_SPST_StandexMeder_SIL_Form1A"
+		(property "Footprint" "UV_Vis_Library:Relay_SPDT_9007_05_00"
 			(at 135.89 86.36 0)
 			(hide yes)
@@
 			)
 		)
-		(property "Footprint" "Relay_THT:Relay_SPST_StandexMeder_SIL_Form1A"
+		(property "Footprint" "UV_Vis_Library:Relay_SPDT_9007_05_00"
 			(at 135.89 104.14 0)
 			(hide yes)

Commit message: Added guard trace.
Connections:
- net SW2: now reaches C1.2, R6.2, RR2.1
- net SW1: now reaches C11.2, R7.2, RR1.1
- net SW3: now reaches C10.2, R5.2, RR3.1
Changed lines of the file:
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@@
+		)
+	)
+	(label "SW1"
+		(at 121.92 78.74 0)
+		(effects
+			(font
+				(size 1.27 1.27)
+			)
+			(justify left bottom)
 		)
 	)
@@
 		(effects
 			(font
+				(size 1.27 1.27)
+			)
+			(justify left bottom)
+		)
+	)
+	(label "SW3"
+		(at 121.92 114.3 0)
+		(effects
+			(font
+				(size 1.27 1.27)
+			)
+			(justify left bottom)
+		)
+	)
+	(label "SW2"
+		(at 121.92 96.52 0)
+		(effects
+			(font
